File: circuit/main2.brd (EAGLE design)
At the start: 21.6 x 20.6 mm, 18 parts, among them IC2 LD398533RM, J1 22-27-2041-04, J2 22-27-2041-04, Q2 BSS138, Q3 12MHz, U1 ATTINY84-20SSU

Commit message: Updated circuit for Shinewave v0.3
Signed-off-by: Garrett Greenwood <garrettagreenwood@gmail.com>
Parts:
- moved R1 7.94 mm to (21.0, 12.4)
- moved R2 7.94 mm to (21.0, 9.84)
- moved R3 6.35 mm to (13.3, 9.84), turned to 0 degrees
- moved R5 5.17 mm to (17.1, 12.7), turned to 180 degrees
- moved C2 4.76 mm to (17.1, 15.2), turned to 180 degrees
- moved C1 3.82 mm to (21.0, 14.9)
- moved R4 3.82 mm to (13.3, 12.4), turned to 180 degrees
- moved IC2 2.31 mm to (21.3, 17.8), turned to 270 degrees
- moved C3 0.45 mm to (13.3, 14.9)
- moved C4 0.32 mm to (7.94, 20.0)
- moved C5 0.32 mm to (7.94, 16.8)
- moved Q3 0.32 mm to (4.45, 18.4)
- moved U1 0.32 mm to (6.99, 11.4)
- moved U$1 0.32 mm to (9.21, 10.5)
- moved U$3 0.32 mm to (14.3, 20.3)
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Connections:
- new net MOSI/GCN_SIG: U$1.MOSI
- net MOSI/SIG1: no longer U$1.MOSI
Routing:
- net 5V: track 52.2 -> 0.00 mm
- net 3.3V: track 43.9 -> 2.72 mm, vias 1 -> 0
- net SIG2: track 17.7 -> 0.00 mm
- net N$1: track 17.3 -> 0.00 mm
- net N$6: track 12.1 -> 0.00 mm
- net USB_D+: track 12.2 -> 1.27 mm
- net USB_D-: track 9.23 -> 0.00 mm
- net GND: track 8.97 -> 0.00 mm, vias 4 -> 0
- net N$5: track 7.21 -> 0.00 mm
- net MOSI/SIG1: track 19.0 -> 12.0 mm
- net N$4: track 2.53 -> 0.00 mm
- net RESET: track 5.64 -> 4.37 mm
- net MISO: track 5.64 -> 6.27 mm
- removed copper zone on layer 1, net GND
- removed copper zone on layer 16, net GND
Other:
- board size 21.6 x 20.6 mm -> 22.2 x 20.6 mm
- board text added: "ATTiny84"
- board text removed: "3.3V"
- board text removed: "5V"
- board text removed: "GND"
- board text removed: "Garrett Greenwood"
- board text removed: "SIG1"
- board text removed: "SIG2"
- board text removed: "Shinewave v0.3"
