File: circuit/main2.sch (EAGLE design)
At the start: 18 parts, among them IC2 LD398533RM, J1 22-27-2041-04, J2 22-27-2041-04, Q2 BSS138, Q3 12MHz, U1 ATTINY84-20SSU

Commit message: Updated circuit for Shinewave v0.3
Signed-off-by: Garrett Greenwood <garrettagreenwood@gmail.com>
Connections:
- new net MOSI/GCN_SIG: U$1.MOSI
- net MOSI/SIG1: no longer U$1.MOSI
Changed lines of the file:
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@@
+</segment>
+</net>
+<net name="MOSI/GCN_SIG" class="0">
+<segment>
+<wire x1="127" y1="116.84" x2="132.08" y2="116.84" width="0.1524" layer="91"/>
+<label x="132.08" y="116.84" size="1.778" layer="95" xref="yes"/>
+<pinref part="U$1" gate="G$1" pin="MOSI"/>
 </segment>
 </net>
@@
 <label x="88.9" y="50.8" size="1.27" layer="95" xref="yes"/>
 </segment>
-<segment>
-<wire x1="127" y1="116.84" x2="132.08" y2="116.84" width="0.1524" layer="91"/>
-<label x="132.08" y="116.84" size="1.778" layer="95" xref="yes"/>
-<pinref part="U$1" gate="G$1" pin="MOSI"/>
-</segment>
 </net>
